File: eagle/WaterLevelIndicator.brd (EAGLE design)
At the start: 58.4 x 81 mm, 7 parts, among them IC2 MAX7219CNG

Commit message: added eagle schematics
Routing:
- net N$14: track 30.5 -> 131.8 mm
- net N$12: track 70.6 -> 0.00 mm
- net N$5: track 67.4 -> 0.00 mm
- net N$27: track 55.4 -> 0.00 mm
- net N$4: track 45.7 -> 0.00 mm
- net N$7: track 32.7 -> 0.00 mm
- net N$1: track 92.3 -> 116.0 mm, vias 1 -> 0
- net N$19: track 33.4 -> 49.8 mm
- net N$26: track 31.2 -> 46.2 mm
- net N$13: track 40.4 -> 52.5 mm
- net N$6: track 96.3 -> 104.9 mm
- net N$18: track 38.0 -> 45.2 mm
- net N$22: track 29.1 -> 36.3 mm
- net N$16: track 15.7 -> 20.7 mm
- net N$23: track 13.9 -> 17.5 mm
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