File: eagle/WaterLevelIndicator.brd (EAGLE design)
At the start: 52 x 75.9 mm, 7 parts, among them IC2 MAX7219CNG

Commit message: current
Parts:
- moved C1 30.7 mm to (17.8, 66.0), turned to 270 degrees
- moved C2 30.7 mm to (29.2, 66.0), turned to 270 degrees
- moved R1 26.4 mm to (22.9, 74.9), turned to 90 degrees
- moved IC2 4.58 mm to (24.1, 87.6), turned to 180 degrees
Connections:
- net N$5: now also U$1.JP1.5; no longer U$1.JP1.7
Routing:
- net N$1: track 0.00 -> 138.2 mm
- net N$13: track 0.00 -> 83.3 mm
- net N$4: track 0.00 -> 60.6 mm
- net N$24: track 0.00 -> 55.0 mm
- net N$28: track 0.00 -> 42.3 mm
- net N$20: track 0.00 -> 41.3 mm
- net N$21: track 0.00 -> 39.5 mm
- net N$17: track 0.00 -> 39.2 mm
- net N$19: track 0.00 -> 36.3 mm
- net N$27: track 0.00 -> 36.1 mm
- net N$22: track 0.00 -> 33.9 mm
- net N$2: track 0.00 -> 32.5 mm
- net N$25: track 0.00 -> 28.6 mm
- net N$15: track 0.00 -> 28.1 mm
- net N$26: track 0.00 -> 20.9 mm
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
Commit message: more optimization
Parts:
- moved U$1 1.27 mm to (15.2, 40.6)
Connections:
- net N$4: now also U$1.JP1.6; no longer U$1.JP1.4
- net N$6: now also U$1.JP1.4; no longer U$1.JP1.6
Routing:
- net N$13: track 83.3 -> 11.5 mm
- net N$23: track 0.00 -> 67.8 mm
- net N$4: track 60.6 -> 112.5 mm
- net N$1: track 138.2 -> 188.4 mm
- net N$14: track 0.00 -> 40.7 mm
- net N$17: track 39.2 -> 0.00 mm
- net N$16: track 0.00 -> 34.2 mm
- net N$18: track 0.00 -> 22.3 mm
- net N$21: track 39.5 -> 17.9 mm
- net N$24: track 55.0 -> 33.5 mm
- net N$27: track 36.1 -> 18.8 mm
- net N$15: track 28.1 -> 44.1 mm
- net N$12: track 0.00 -> 14.1 mm
- net N$28: track 42.3 -> 30.7 mm
- net N$26: track 20.9 -> 32.1 mm
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Other:
- board size 52 x 75.9 mm -> 58.4 x 78.4 mm

Commit message: add holes
Routing:
- net N$5: track 0.00 -> 38.9 mm, vias 0 -> 1
- net N$6: track 0.00 -> 31.3 mm
- net N$4: track 112.5 -> 120.1 mm
- net N$1: track 188.4 -> 185.3 mm
- net N$17: track 0.00 -> 1.66 mm
- net N$16: track 34.2 -> 35.4 mm
Other:
- board size 58.4 x 78.4 mm -> 54.6 x 77.1 mm
Changed lines of the file:
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@@
 <layer number="43" name="vRestrict" color="2" fill="10" visible="yes" active="yes"/>
 <layer number="44" name="Drills" color="7" fill="1" visible="no" active="yes"/>
-<layer number="45" name="Holes" color="7" fill="1" visible="no" active="yes"/>
+<layer number="45" name="Holes" color="7" fill="1" visible="yes" active="yes"/>
 <layer number="46" name="Milling" color="3" fill="1" visible="no" active="yes"/>
 <layer number="47" name="Measures" color="7" fill="1" visible="no" active="yes"/>
@@
 <board>
 <plain>
-<wire x1="-3.81" y1="24.13" x2="54.59" y2="24.13" width="0" layer="20"/>
-<wire x1="54.59" y1="24.13" x2="54.59" y2="102.54" width="0" layer="20"/>
-<wire x1="54.59" y1="102.54" x2="-3.81" y2="102.54" width="0" layer="20"/>
-<wire x1="-3.81" y1="102.54" x2="-3.81" y2="24.13" width="0" layer="20"/>
+<wire x1="-2.54" y1="24.13" x2="52.05" y2="24.13" width="0" layer="20"/>
+<wire x1="52.05" y1="24.13" x2="52.05" y2="101.27" width="0" layer="20"/>
+<wire x1="52.05" y1="101.27" x2="-2.54" y2="101.27" width="0" layer="20"/>
+<wire x1="-2.54" y1="101.27" x2="-2.54" y2="24.13" width="0" layer="20"/>
 </plain>
 <attributes>
@@
 <wire x1="23.495" y1="64.77" x2="17.78" y2="64.77" width="0.254" layer="1"/>
 <wire x1="29.21" y1="64.77" x2="29.21" y2="65.024" width="0.254" layer="1"/>
-<wire x1="10.16" y1="99.06" x2="17.78" y2="91.44" width="0.254" layer="1"/>
 <wire x1="1.27" y1="99.06" x2="10.16" y2="99.06" width="0.254" layer="1"/>
 <wire x1="-1.27" y1="96.52" x2="1.27" y2="99.06" width="0.254" layer="1"/>
@@
 <wire x1="50.165" y1="98.425" x2="50.165" y2="97.155" width="0.254" layer="1"/>
 <wire x1="49.53" y1="99.06" x2="50.165" y2="98.425" width="0.254" layer="1"/>
-<wire x1="10.16" y1="99.06" x2="49.53" y2="99.06" width="0.254" layer="1"/>
+<wire x1="10.16" y1="99.06" x2="17.78" y2="99.06" width="0.254" layer="1"/>
+<wire x1="17.78" y1="99.06" x2="49.53" y2="99.06" width="0.254" layer="1"/>
 <wire x1="23.495" y1="64.77" x2="32.385" y2="55.88" width="0.254" layer="1"/>
 <wire x1="32.385" y1="55.88" x2="32.94" y2="55.34" width="0.254" layer="1"/>
+<wire x1="17.78" y1="91.44" x2="17.78" y2="99.06" width="0.254" layer="1"/>
 </signal>
 <signal name="N$2">
@@
 <wire x1="50.165" y1="90.805" x2="49.53" y2="91.44" width="0.254" layer="1"/>
 <wire x1="50.165" y1="86.995" x2="50.165" y2="90.805" width="0.254" layer="1"/>
-<wire x1="49.53" y1="86.36" x2="50.165" y2="86.995" width="0.254" layer="1"/>
-<wire x1="47.625" y1="86.36" x2="49.53" y2="86.36" width="0.254" layer="1"/>
-<wire x1="46.99" y1="85.725" x2="47.625" y2="86.36" width="0.254" layer="1"/>
-<wire x1="46.99" y1="81.915" x2="46.99" y2="85.725" width="0.254" layer="1"/>
-<wire x1="47.625" y1="81.28" x2="46.99" y2="81.915" width="0.254" layer="1"/>
-<wire x1="49.53" y1="81.28" x2="47.625" y2="81.28" width="0.254" layer="1"/>
-<wire x1="50.165" y1="80.645" x2="49.53" y2="81.28" width="0.254" layer="1"/>
+<wire x1="50.165" y1="86.995" x2="49.53" y2="86.36" width="0.254" layer="1"/>
+<wire x1="49.53" y1="81.28" x2="50.165" y2="80.645" width="0.254" layer="1"/>
 <wire x1="50.165" y1="53.975" x2="50.165" y2="80.645" width="0.254" layer="1"/>
 <wire x1="27.305" y1="31.115" x2="50.165" y2="53.975" width="0.254" layer="1"/>
 <wire x1="10.16" y1="31.115" x2="27.305" y2="31.115" width="0.254" layer="1"/>
 <wire x1="3.81" y1="37.465" x2="10.16" y2="31.115" width="0.254" layer="1"/>
+<wire x1="43.18" y1="86.36" x2="43.18" y2="82.55" width="0.254" layer="1"/>
+<wire x1="43.18" y1="82.55" x2="44.45" y2="81.28" width="0.254" layer="1"/>
+<wire x1="49.53" y1="86.36" x2="43.18" y2="86.36" width="0.254" layer="1"/>
+<wire x1="44.45" y1="81.28" x2="49.53" y2="81.28" width="0.254" layer="1"/>
 </signal>
 <signal name="N$5">
 <contactref element="IC2" pad="12"/>
 <contactref element="U$1" pad="JP1.5"/>
-<wire x1="3.81" y1="40.005" x2="10.16" y2="91.44" width="0" layer="19" extent="1-1"/>
+<wire x1="10.16" y1="91.44" x2="7.62" y2="91.44" width="0.254" layer="1"/>
+<wire x1="3.81" y1="40.005" x2="-0.635" y2="40.005" width="0.254" layer="1"/>
+<wire x1="-0.635" y1="40.005" x2="-1.27" y2="40.64" width="0.254" layer="1"/>
+<wire x1="-1.27" y1="40.64" x2="-1.27" y2="68.58" width="0.254" layer="1"/>
+<wire x1="-1.27" y1="68.58" x2="0" y2="69.85" width="0.254" layer="1"/>
+<wire x1="0" y1="69.85" x2="1.27" y2="69.85" width="0.254" layer="1"/>
+<via x="1.27" y="69.85" extent="1-16" drill="1" shape="square"/>
+<wire x1="1.27" y1="69.85" x2="7.62" y2="91.44" width="0" layer="19" extent="1-1"/>
 </signal>
 <signal name="N$6">
 <contactref element="IC2" pad="13"/>
 <contactref element="U$1" pad="JP1.4"/>
-<wire x1="3.81" y1="42.545" x2="10.16" y2="83.82" width="0" layer="19" extent="1-1"/>
+<wire x1="3.81" y1="42.545" x2="0.635" y2="42.545" width="0.254" layer="1"/>
+<wire x1="0.635" y1="42.545" x2="0" y2="43.18" width="0.254" layer="1"/>
+<wire x1="0" y1="43.18" x2="0" y2="66.04" width="0.254" layer="1"/>
+<wire x1="10.16" y1="83.82" x2="8.89" y2="83.82" width="0.254" layer="1"/>
+<wire x1="8.89" y1="83.82" x2="7.62" y2="85.09" width="0.254" layer="1"/>
+<wire x1="7.62" y1="85.09" x2="7.62" y2="86.36" width="0.254" layer="1"/>
+<wire x1="0" y1="66.04" x2="10.16" y2="83.82" width="0" layer="19" extent="1-1"/>
 </signal>
 <signal name="N$7">
@@
 <wire x1="50.8" y1="85.09" x2="48.895" y2="83.185" width="0.254" layer="1"/>
 <wire x1="50.8" y1="92.71" x2="50.8" y2="85.09" width="0.254" layer="1"/>
-<wire x1="49.53" y1="93.98" x2="50.8" y2="92.71" width="0.254" layer="1"/>
-<wire x1="33.02" y1="93.98" x2="49.53" y2="93.98" width="0.254" layer="1"/>
+<wire x1="50.8" y1="92.71" x2="49.53" y2="93.98" width="0.254" layer="1"/>
+<wire x1="49.53" y1="93.98" x2="33.02" y2="93.98" width="0.254" layer="1"/>
 <wire x1="31.75" y1="92.71" x2="33.02" y2="93.98" width="0.254" layer="1"/>
 <wire x1="31.75" y1="90.17" x2="31.75" y2="92.71" width="0.254" layer="1"/>
@@
 <contactref element="IC2" pad="3"/>
 <contactref element="U$3" pad="P$6"/>
-<wire x1="13.335" y1="85.725" x2="2.54" y2="85.725" width="0.254" layer="1"/>
-<wire x1="15.875" y1="88.265" x2="13.335" y2="85.725" width="0.254" layer="1"/>
 <wire x1="31.115" y1="88.265" x2="15.875" y2="88.265" width="0.254" layer="1"/>
 <wire x1="33.02" y1="90.17" x2="31.115" y2="88.265" width="0.254" layer="1"/>
 <wire x1="33.02" y1="91.44" x2="33.02" y2="90.17" width="0.254" layer="1"/>
-<wire x1="2.54" y1="85.725" x2="2.2" y2="85.24" width="0.254" layer="1"/>
+<wire x1="2.2" y1="85.24" x2="3.96" y2="85.24" width="0.254" layer="1"/>
+<wire x1="3.96" y1="85.24" x2="5.08" y2="86.36" width="0.254" layer="1"/>
+<wire x1="5.08" y1="86.36" x2="5.08" y2="87.63" width="0.254" layer="1"/>
+<wire x1="5.08" y1="87.63" x2="6.35" y2="88.9" width="0.254" layer="1"/>
+<wire x1="15.24" y1="88.9" x2="15.875" y2="88.265" width="0.254" layer="1"/>
+<wire x1="6.35" y1="88.9" x2="15.24" y2="88.9" width="0.254" layer="1"/>
 </signal>
 <signal name="N$17">
 <contactref element="IC2" pad="10"/>
 <contactref element="U$3" pad="P$11"/>
-<wire x1="15.24" y1="91.44" x2="48.63" y2="85.14" width="0" layer="19" extent="1-1"/>
+<wire x1="48.63" y1="85.14" x2="48.58" y2="85.09" width="0.254" layer="1"/>
+<wire x1="48.58" y1="85.09" x2="46.99" y2="85.09" width="0.254" layer="1"/>
+<wire x1="15.24" y1="91.44" x2="46.99" y2="85.09" width="0" layer="19" extent="1-1"/>
 </signal>
 <signal name="N$18">
@@
 <wire x1="25.4" y1="67.31" x2="25.4" y2="83.82" width="0.6096" layer="1"/>
 </signal>
+<signal name="N$8">
+<via x="1.27" y="66.04" extent="1-16" drill="1" shape="square"/>
+</signal>
 </signals>

Commit message: changes
Connections:
- removed net N$3: U$1.JP1.8
- net N$28: now also U$1.JP1.8
- net N$4: now also U$1.JP2.6; no longer U$1.JP1.6
Routing:
- net N$24: track 33.5 -> 117.4 mm
- net N$1: track 185.3 -> 103.9 mm
- net N$17: track 1.66 -> 53.3 mm
- net N$4: track 120.1 -> 76.9 mm
- net N$20: track 41.7 -> 0.00 mm
- net N$28: track 30.7 -> 71.4 mm
- net N$16: track 35.4 -> 0.00 mm
- net N$6: track 31.3 -> 65.5 mm
- net N$5: track 38.9 -> 70.1 mm, vias 1 -> 0
- net N$23: track 67.8 -> 87.6 mm
- net N$22: track 25.3 -> 35.9 mm
- net N$25: track 32.6 -> 22.1 mm
- net N$15: track 44.1 -> 48.9 mm
- net N$19: track 31.7 -> 34.0 mm
- net N$14: track 40.7 -> 38.9 mm
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Other:
- board size 54.6 x 77.1 mm -> 62.2 x 78.4 mm
